File: KiCAD/Keyboard-MC7007-Short.kicad_pcb (KiCad board)
At the start: 2 copper layers, 298.6 x 137.5 mm, 90 parts

Commit message: v1.0.2
Parts:
- moved S75 7.13 mm to (215.7, 129.7)
- moved STAB_7 7.13 mm to (244.2, 148.7)
- moved S4 7.12 mm to (244.2, 148.7)
- moved S76 7.12 mm to (272.7, 148.7)
- moved S44 7.12 mm to (139.7, 129.7)
- moved S51 7.12 mm to (158.7, 129.7)
- moved S60 7.12 mm to (177.7, 129.7)
- moved S84 7.12 mm to (253.7, 129.7)
- moved S11 7.12 mm to (63.7, 129.7)
- moved S19 7.12 mm to (82.7, 129.7)
- moved S28 7.12 mm to (101.7, 129.7)
- moved S36 7.12 mm to (120.7, 129.7)
- moved S61 7.12 mm to (291.7, 148.7)
- moved S62 7.12 mm to (291.7, 129.7)
- moved S68 7.12 mm to (196.7, 129.7)
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Routing:
- net /ROW5: track 418.1 -> 425.8 mm
- net /COL1: track 447.8 -> 454.3 mm
- net /COL8: track 469.1 -> 464.1 mm
- net /COL10: track 245.8 -> 241.9 mm
- net /ROW3: track 408.0 -> 404.3 mm
- net /COL6: track 347.4 -> 344.4 mm
- net /COL7: track 354.7 -> 352.0 mm
- net /ROW6: track 311.9 -> 309.5 mm
- net /COL2: track 224.4 -> 222.4 mm
- net /COL11: track 172.9 -> 170.9 mm
- net /COL5: track 325.5 -> 323.5 mm
- net /COL4: track 235.2 -> 233.2 mm
- net /ROW4: track 319.2 -> 317.7 mm
- net /ROW7: track 274.5 -> 275.9 mm
- net /ROW8: track 227.7 -> 226.8 mm
Other:
- board text added: "Off center"
